Commit message: update urdf; Cartesican spcace control

File: otter/gym/bullet/assets/urdf/j2s7s300.urdf (robot description, URDF)
Before this commit: robot j2s7s300, 17 links, 16 joints
Joints:
- joint j2s7s300_joint_1: limit lower=-6.28318530718 upper=6.28318530718 effort=2000 velocity=1 -> lower=-18.849555921540002 upper=18.849555921540002 effort=2000 velocity=1
- joint j2s7s300_joint_3: limit lower=-6.28318530718 upper=6.28318530718 effort=2000 velocity=1 -> lower=-18.849555921540002 upper=18.849555921540002 effort=2000 velocity=1
- joint j2s7s300_joint_5: limit lower=-6.28318530718 upper=6.28318530718 effort=2000 velocity=1 -> lower=-18.849555921540002 upper=18.849555921540002 effort=2000 velocity=1
- joint j2s7s300_joint_7: limit lower=-6.28318530718 upper=6.28318530718 effort=2000 velocity=1 -> lower=-18.849555921540002 upper=18.849555921540002 effort=2000 velocity=1
