Commit message: framework

File: otter/gym/bullet/assets/urdf/TeaCup.urdf (robot description, URDF)
Before this commit: robot TeaCup, 1 links, 0 joints
Links:
- link TeaCupLink: mass 1.0 -> 0.15; geometry collision mesh filename=TeaCup.obj scale=0.01 0.01 0.01; visual mesh filename=TeaCup.obj scale=0.04 0.04 0.04

File: otter/gym/bullet/assets/urdf/coffee_cup.urdf (robot description, URDF)
Before this commit: robot TeaCup, 1 links, 0 joints
Links:
- link TeaCupLink: mass None -> 0.15; geometry collision mesh filename=coffee_cup.obj scale=0.02 0.02 0.02; visual mesh filename=coffee_cup.obj scale=0.02 0.02 0.02
